Commit message: Add linked model

File: urdf/simeon_2004.urdf (robot description, URDF)
Before this commit: robot simeon_2004, 1 links, 0 joints
Links:
- added link blocks; collision box size=1.0 1.0 0.3; collision box size=3.0 0.3 0.3
- added link cage_bars; collision mesh filename=../meshes/dae/lattice_bar_geometry.dae scale=0.40575 0.40575 0.40575; collision mesh filename=../meshes/dae/lattice_bar_geometry.dae scale=0.40575 0.40575 0.40575
- added link object, mass 1.0; collision box size=2.0 0.16 0.16; visual box size=2.0 0.16 0.16
- link floor: geometry collision box size=9.04809 9.04809 0; visual box size=9.04809 9.04809 0
Joints:
- added joint blocks: type fixed, parent floor, child blocks, origin xyz=1.03374 0.48892 0.30001 rpy=0 0 0
- added joint cage_bars: type floating, parent floor, child cage_bars, origin xyz=0.85774 0.60024 0 rpy=0 0 0
- added joint object: type floating, parent floor, child object, origin xyz=0.85774 -1.40834 0.03 rpy=0 0 0, limit effort=0 velocity=0

Commit message: Fix files

File: urdf/simeon_2004.urdf (robot description, URDF)
Before this commit: robot simeon_2004, 4 links, 3 joints
Links:
- removed link object
- added link obj1, mass 1.0; collision box size=2.0 0.16 0.16; visual box size=2.0 0.16 0.16
Joints:
- removed joint object
- added joint obj1: type floating, parent floor, child obj1, origin xyz=0.85774 -1.40834 0.03 rpy=0 0 0, limit effort=0 velocity=0
