Commit message: Clean up conversion scripts

File: models/simeon_2004/simeon_2004.urdf (robot description, URDF)
Before this commit: robot simeon_2004, 4 links, 3 joints
Links:
- link cage_bars: geometry collision mesh filename=meshes/dae/lattice_bar_geometry.dae scale=0.40575 0.40575 0.40575; collision mesh filename=meshes/dae/lattice_bar_geometry.dae scale=0.40575 0.40575 0.40575
